File: eagle/mult.brd (EAGLE design)
At the start: 100.6 x 81.3 mm, 18 parts, among them IC1 TL074P

Commit message: starting the panel
Parts:
- added R6: 10k, rcl:0207/10
- moved R2 0.64 mm to (18.4, 41.9)
- moved C3 0.63 mm to (26.7, 23.5)
Connections:
- new net N$6: INPUT.P$2, R6.2
- net GND: now also R6.1; no longer INPUT.P$2
Routing:
- net GND: track 185.3 -> 167.4 mm
- net N$12: track 67.0 -> 51.8 mm
- net N$6: track 0.00 -> 5.07 mm
- net N$2: track 8.93 -> 7.82 mm
- net N$3: track 7.29 -> 6.66 mm
- net N$7: track 8.45 -> 8.97 mm
Other:
- outline, holes or cut-outs redrawn
